Commit message: Ejemplo uso de sensores funcionando

File: my_robot_description/urdf/my_robot.urdf (robot description, URDF)
Before this commit: robot my_robot, 5 links, 4 joints
Links:
- added link camera_link, mass 0.1; collision box size=0.01 0.1 0.05; visual box size=0.01 0.1 0.05
Joints:
- added joint base_camera_joint: type fixed, parent base_link, child camera_link, origin xyz=0.305 0 0.1 rpy=0 0 0

File: my_robot_description/urdf/my_robot.urdf.xacro (robot description, xacro)
@@ -3,3 +3,4 @@
     <xacro:include filename="common_properties.xacro"/>
     <xacro:include filename="mobile_base.xacro"/>
+    <xacro:include filename="camera.xacro"/>
 </robot>
