Commit message: arm sin acoplarlo al robot

File: my_robot_description/urdf/common_properties.xacro (robot description, xacro)
@@ -6,4 +6,10 @@
     <material name="grey">
         <color rgba="0.5 0.5 0.5 1"/>
+    </material>
+    <material name="orange">
+        <color rgba="1 0.5 0 1"/>
+    </material>
+    <material name="yellow">
+        <color rgba="1 1 0 1"/>
     </material>
     <xacro:macro name="box_inertia" params="m l w h xyz rpy">
