Commit message: arm integrado Rviz ok

File: my_robot_description/urdf/arm.xacro (robot description, xacro)
@@ -16,4 +16,11 @@
             <material name="orange"/>
         </visual>
+        <collision>
+            <geometry>
+                <box size="${arm_base_length} ${arm_base_width} ${arm_base_height}"/>
+            </geometry>
+            <origin xyz="0 0 ${arm_base_height/2.0}" rpy="0 0 0"/>
+        </collision>
+        <xacro:box_inertia m="0.5" l="${arm_base_length}" w="${arm_base_width}" h="${arm_base_height}" xyz="0 0 ${arm_base_height/2.0}" rpy="0 0 0"/>
     </link>
     <link name="forearm_link">
@@ -25,4 +32,11 @@
             <material name="yellow"/>
         </visual>
+        <collision>
+            <geometry>
+                <cylinder radius="${forearm_radius}" length="${forearm_length}"/>
+            </geometry>
+            <origin xyz="0 0 ${forearm_length/2.0}" rpy="0 0 0"/>
+        </collision>
+        <xacro:cylinder_inertia m="0.3" r="${forearm_radius}" h="${forearm_length}" xyz="0 0 ${forearm_length/2.0}" rpy="0 0 0"/>
     </link>
     <link name="hand_link">
@@ -34,4 +48,11 @@
             <material name="orange"/>
         </visual>
+        <collision>
+            <geometry>
+                <cylinder radius="${hand_radius}" length="${hand_length}"/>
+            </geometry>
+            <origin xyz="0 0 ${hand_length/2.0}" rpy="0 0 0"/>
+        </collision>
+        <xacro:cylinder_inertia m="0.3" r="${hand_radius}" h="${hand_length}" xyz="0 0 ${hand_length/2.0}" rpy="0 0 0"/>
     </link>
     <joint name="arm_base_forearm_joint" type="revolute">

File: my_robot_description/urdf/mobile_base.xacro (robot description, xacro)
@@ -90,3 +90,8 @@
         <origin xyz="0 0 ${wheel_radius}" rpy="0 0 0"/>
     </joint>
+    <joint name="mobile_base_arm_base_joint" type="fixed">
+        <parent link="base_link"/>
+        <child link="arm_base_link"/>
+        <origin xyz="${base_length/3.5} 0 ${base_height}" rpy="0 0 ${pi/2.0}"/>
+    </joint>
 </robot>

File: my_robot_description/urdf/my_robot.urdf.xacro (robot description, xacro)
@@ -2,4 +2,5 @@
 <robot name="my_robot" xmlns:xacro="http://www.ros.org/wiki/xacro">
     <xacro:include filename="common_properties.xacro"/>
+    <xacro:include filename="arm.xacro"/>
     <xacro:include filename="mobile_base.xacro"/>
     <xacro:include filename="camera.xacro"/>

Commit message: final project terminado en ignition

File: my_robot_description/urdf/arm.xacro (robot description, xacro)
@@ -61,4 +61,5 @@
         <origin xyz="0 0 ${arm_base_height}" rpy="0 0 0"/>
         <limit lower="0" upper="${pi/2}" effort="100" velocity="100"/>
+        <dynamics friction="0.05" damping="0.1"/>
     </joint>
     <joint name="forearm_hand_joint" type="revolute">
@@ -67,4 +68,5 @@
         <origin xyz="0 0 ${forearm_length}" rpy="0 0 0"/>
         <limit lower="0" upper="${pi/2}" effort="100" velocity="100"/>
+        <dynamics friction="0.05" damping="0.1"/>
     </joint>
 </robot>
